Commit message: 修复 tf, 调整 nav2 参数,修改 lidarscan

File: src/rm_vision/rm_description/urdf/sentry.urdf.xacro (robot description, xacro)
@@ -6,4 +6,5 @@
   <link name="chassis"/>
   <joint name="base_to_chassis" type="fixed">
+    <origin xyz="0 0 0" rpy="0 0 0" />
     <parent link="base_link" />
     <child link="chassis" />
@@ -11,7 +12,7 @@
   <!-- 云台部分 -->
   <link name="gimbal_odom" />
-  <joint name="gimbal_joint" type="fixed">
-    <origin xyz="0 0 0.2" rpy="0 0 0" />
-    <parent link="base_link" />
+  <joint name="gimbal_joint" type="continuous">
+    <origin xyz="0 0 0.35" rpy="0 0 0" />
+    <parent link="chassis" />
     <child link="gimbal_odom" />
   </joint>
@@ -24,5 +25,5 @@
   <link name="livox_frame"/>
   <joint name="yaw_to_livox" type="fixed">
-    <origin xyz="0 0.07 0.2" rpy="0 0 0" />
+    <origin xyz="-0.03 0.117 0" rpy="0 0 0" />
     <parent link="yaw_link"/>
     <child link="livox_frame" />

Commit message: 修好 gicp 的 initpose 问题

File: src/rm_vision/rm_description/urdf/sentry.urdf.xacro (robot description, xacro)
@@ -12,5 +12,5 @@
   <!-- 云台部分 -->
   <link name="gimbal_odom" />
-  <joint name="gimbal_joint" type="continuous">
+  <joint name="gimbal_joint" type="fixed">
     <origin xyz="0 0 0.35" rpy="0 0 0" />
     <parent link="chassis" />
@@ -18,5 +18,6 @@
   </joint>
   <link name="yaw_link" />
-  <joint name="yaw_joint" type="continuous">
+  <joint name="yaw_joint" type="fixed">
+    <origin xyz="0 0 0.35" rpy="0 0 0" />
     <parent link="gimbal_odom" />
     <child link="yaw_link" />

Commit message: 暂存

File: src/rm_vision/rm_description/urdf/sentry.urdf.xacro (robot description, xacro)
@@ -4,4 +4,5 @@
   <!-- 底盘部分 -->
   <link name="base_link" />
+  <!-- 底盘连接 - 与serial_driver中的base_to_chassis TF对应 -->
   <link name="chassis"/>
   <joint name="base_to_chassis" type="fixed">
@@ -10,24 +11,27 @@
     <child link="chassis" />
   </joint>
-  <!-- 云台部分 -->
+  <!-- 云台odom连接 - 与serial_driver中的chassis_to_gimbal TF对应 -->
   <link name="gimbal_odom" />
-  <joint name="gimbal_joint" type="fixed">
+  <joint name="chassis_to_gimbal" type="continuous">
     <origin xyz="0 0 0.35" rpy="0 0 0" />
     <parent link="chassis" />
     <child link="gimbal_odom" />
+    <axis xyz="0 0 1" />
   </joint>
+  <!-- 云台yaw轴 -->
   <link name="yaw_link" />
-  <joint name="yaw_joint" type="fixed">
-    <origin xyz="0 0 0.35" rpy="0 0 0" />
+  <joint name="yaw_joint" type="continuous">
     <parent link="gimbal_odom" />
     <child link="yaw_link" />
     <axis xyz="0 0 1" />
   </joint>
+  <!-- 激光雷达连接 -->
   <link name="livox_frame"/>
   <joint name="yaw_to_livox" type="fixed">
-    <origin xyz="-0.03 0.117 0" rpy="0 0 0" />
+    <origin xyz="0 0.07 0.2" rpy="0 0 0" />
     <parent link="yaw_link"/>
     <child link="livox_frame" />
   </joint>
+  <!-- 云台pitch轴 -->
   <link name="pitch_link" />
   <joint name="pitch_joint" type="continuous">
@@ -36,4 +40,5 @@
     <axis xyz="0 -1 0" />
   </joint>
+  <!-- 相机连接 -->
   <link name="camera_link" />
   <joint name="camera_joint" type="fixed">

Commit message: 233

File: src/rm_vision/rm_description/urdf/sentry.urdf.xacro (robot description, xacro)
@@ -4,5 +4,4 @@
   <!-- 底盘部分 -->
   <link name="base_link" />
-  <!-- 底盘连接 - 与serial_driver中的base_to_chassis TF对应 -->
   <link name="chassis"/>
   <joint name="base_to_chassis" type="fixed">
@@ -11,13 +10,11 @@
     <child link="chassis" />
   </joint>
-  <!-- 云台odom连接 - 与serial_driver中的chassis_to_gimbal TF对应 -->
+  <!-- 云台部分 -->
   <link name="gimbal_odom" />
-  <joint name="chassis_to_gimbal" type="continuous">
+  <joint name="gimbal_joint" type="continuous">
     <origin xyz="0 0 0.35" rpy="0 0 0" />
     <parent link="chassis" />
     <child link="gimbal_odom" />
-    <axis xyz="0 0 1" />
   </joint>
-  <!-- 云台yaw轴 -->
   <link name="yaw_link" />
   <joint name="yaw_joint" type="continuous">
@@ -26,12 +23,10 @@
     <axis xyz="0 0 1" />
   </joint>
-  <!-- 激光雷达连接 -->
   <link name="livox_frame"/>
   <joint name="yaw_to_livox" type="fixed">
-    <origin xyz="0 0.07 0.2" rpy="0 0 0" />
+    <origin xyz="-0.03 0.117 0" rpy="0 0 0" />
     <parent link="yaw_link"/>
     <child link="livox_frame" />
   </joint>
-  <!-- 云台pitch轴 -->
   <link name="pitch_link" />
   <joint name="pitch_joint" type="continuous">
@@ -40,5 +35,4 @@
     <axis xyz="0 -1 0" />
   </joint>
-  <!-- 相机连接 -->
   <link name="camera_link" />
   <joint name="camera_joint" type="fixed">

Commit message: mac

File: src/rm_vision/rm_description/urdf/sentry.urdf.xacro (robot description, xacro)
@@ -18,5 +18,5 @@
   </joint>
   <link name="yaw_link" />
-  <joint name="yaw_joint" type="fixed">
+  <joint name="yaw_joint" type="continuous">
     <origin xyz="0 0 0.35" rpy="0 0 0" />
     <parent link="gimbal_odom" />

Commit message: mac

File: src/rm_vision/rm_description/urdf/sentry.urdf.xacro (robot description, xacro)
@@ -19,4 +19,8 @@
   <link name="yaw_link" />
   <joint name="yaw_joint" type="continuous">
+<<<<<<< HEAD
+=======
+    <origin xyz="0 0 0.35" rpy="0 0 0" />
+>>>>>>> a746979 (mac)
     <parent link="gimbal_odom" />
     <child link="yaw_link" />

Commit message: 第一次

File: src/rm_vision/rm_description/urdf/sentry.urdf.xacro (robot description, xacro)
@@ -13,20 +13,20 @@
   <link name="gimbal_odom" />
   <joint name="gimbal_joint" type="continuous">
-    <origin xyz="0 0 0.35" rpy="0 0 0" />
+    <origin xyz="0 0 0" rpy="0 0 0" />
     <parent link="chassis" />
     <child link="gimbal_odom" />
   </joint>
+  <link name="livox_frame"/>
+  <joint name="yaw_to_livox" type="fixed">
+    <origin xyz="-0.03 0.117 0.15" rpy="0 0 0" />
+    <parent link="gimbal_odom"/>
+    <child link="livox_frame" />
+  </joint>
   <link name="yaw_link" />
   <joint name="yaw_joint" type="continuous">
-    <origin xyz="0 0 0.35" rpy="0 0 0" />
+    <origin xyz="0 0 0" rpy="0 0 0" />
     <parent link="gimbal_odom" />
     <child link="yaw_link" />
     <axis xyz="0 0 1" />
-  </joint>
-  <link name="livox_frame"/>
-  <joint name="yaw_to_livox" type="fixed">
-    <origin xyz="-0.03 0.117 0" rpy="0 0 0" />
-    <parent link="yaw_link"/>
-    <child link="livox_frame" />
   </joint>
   <link name="pitch_link" />
@@ -38,5 +38,5 @@
   <link name="camera_link" />
   <joint name="camera_joint" type="fixed">
-    <origin xyz="0.17 0 0.08" rpy="0 0 0" />
+    <origin xyz="0.17 0 0.00" rpy="0 0 0" />
     <parent link="pitch_link" />
     <child link="camera_link" />

Commit message: uc完全体,嘎嘎乱杀

File: src/rm_vision/rm_description/urdf/sentry.urdf.xacro (robot description, xacro)
@@ -17,10 +17,4 @@
     <child link="gimbal_odom" />
   </joint>
-  <link name="livox_frame"/>
-  <joint name="yaw_to_livox" type="fixed">
-    <origin xyz="-0.03 0.117 0.15" rpy="0 0 0" />
-    <parent link="gimbal_odom"/>
-    <child link="livox_frame" />
-  </joint>
   <link name="yaw_link" />
   <joint name="yaw_joint" type="continuous">
@@ -29,4 +23,10 @@
     <child link="yaw_link" />
     <axis xyz="0 0 1" />
+  </joint>
+  <link name="livox_frame"/>
+  <joint name="yaw_to_livox" type="fixed">
+    <origin xyz="-0.03 0.117 0" rpy="0 0 0" />
+    <parent link="yaw_link"/>
+    <child link="livox_frame" />
   </joint>
   <link name="pitch_link" />
